File: PCBs/spdif_PMOD/spdif_PMOD.kicad_pcb (KiCad board)
At the start: 2 copper layers, 11 parts, among them J1 Conn_01x06_Male, J2 Conn_01x04_Male, J3 Conn_Coaxial, U1 74HC04

Commit message: agrego PCB spdif_pmod terminado
Parts:
- removed J2: Conn_01x04_Male, Connector_PinHeader_2.54mm:PinHeader_1x04_P2.54mm_Vertical
- removed U1: 74HC04, Package_DIP:DIP-14_W7.62mm_LongPads
- added U2: 74HC04, Package_DIP:DIP-14_W7.62mm_LongPads, F.Cu at (193.0, 66.0)
- J3: footprint Connector_Coaxial:BNC_PanelMountable_Vertical -> Connector_BarrelJack:BarrelJack_CUI_PJ-063AH_Horizontal
- moved R3 113.0 mm to (198.1, 87.0), turned to 180 degrees
- moved R2 107.3 mm to (198.8, 61.0)
- moved R1 107.2 mm to (188.0, 61.0)
- moved C3 95.4 mm to (188.6, 71.8), turned to 270 degrees
- moved J3 94.4 mm to (197.5, 56.5), turned to 180 degrees
- moved C2 93.2 mm to (200.7, 90.2), turned to 270 degrees
- moved D1 87.3 mm to (203.2, 85.7), turned to 270 degrees
- moved C1 66.8 mm to (196.2, 90.2), turned to 270 degrees
- moved J1 43.2 mm to (203.2, 97.2), turned to 270 degrees
Connections:
- J1 pad 6: (no net) -> Net-(J1-Pad6)
Routing:
- net GND: track 0.00 -> 105.5 mm
- net +3V3: track 0.00 -> 45.9 mm
- net Net-(J1-Pad5): track 0.00 -> 36.5 mm
- net Net-(C3-Pad2): track 0.00 -> 14.8 mm
- net Net-(C3-Pad1): track 0.00 -> 11.1 mm
- net Net-(J3-Pad1): track 0.00 -> 8.15 mm
- net Net-(D1-Pad1): track 0.00 -> 5.98 mm
- added copper zone on B.Cu, net GND
Other:
- board outline added: 22.9 x 52.1 mm
